Commit message: camera in gazebo sim working

File: src/my_bot/description/robot.urdf.xacro (robot description, xacro)
@@ -4,4 +4,5 @@
     <xacro:arg name="sim_mode" default="false"/>
     <xacro:include filename="robot_core.xacro" />
+    <xacro:include filename="camera.xacro" />
     <xacro:if value="$(arg use_ros2_control)">
         <xacro:include filename="ros2_control.xacro" />

File: src/my_bot/description/robot_core.xacro (robot description, xacro)
@@ -27,4 +27,7 @@
     <material name="black">
         <color rgba="0 0 0 1"/>
+    </material>
+    <material name="red">
+        <color rgba="1 0 0 1"/>
     </material>
     <link name="base_link">
