Commit message: tunned robot params

File: src/my_bot/description/robot_core.xacro (robot description, xacro)
@@ -6,9 +6,9 @@
     <xacro:property name="chassis_height" value="0.046"/>
     <xacro:property name="chassis_mass" value="1.0"/>
-    <xacro:property name="wheel_radius" value="0.034"/>
+    <xacro:property name="wheel_radius" value="0.033"/>
     <xacro:property name="wheel_thickness" value="0.026"/>
     <xacro:property name="wheel_mass" value="0.05"/>
     <xacro:property name="wheel_offset_x" value="0.148"/>
-    <xacro:property name="wheel_offset_y" value="0.092"/>
+    <xacro:property name="wheel_offset_y" value="0.087"/>
     <xacro:property name="wheel_offset_z" value="-0.02"/>
     <xacro:property name="caster_wheel_radius" value="0.01"/>

File: src/my_bot/description/ros2_control.xacro (robot description, xacro)
@@ -34,5 +34,5 @@
                 <param name="baud_rate">57600</param>
                 <param name="timeout_ms">1000</param>
-                <param name="enc_counts_per_rev">675</param>
+                <param name="enc_counts_per_rev">680</param>
                 <param name="pid_p">20</param>
                 <param name="pid_d">12</param>

Commit message: Added nav2 simulation and lidar launch file

File: src/my_bot/description/robot_core.xacro (robot description, xacro)
@@ -32,4 +32,12 @@
     </material>
     <link name="base_link">
+    </link>
+    <!-- BASE_FOOTPRINT -->
+    <joint name="base_footprint_joint" type="fixed">
+        <parent link="base_link"/>
+        <child link="base_footprint"/>
+        <origin xyz="0 0 0" rpy="0 0 0"/>
+    </joint>
+    <link name="base_footprint">
     </link>
     <!-- CHASSIS -->
